File: xmas_2021.kicad_pcb (KiCad board)
At the start: 2 copper layers, 41.4 x 69.4 mm, 36 parts, among them J1 SWIM, SW1 User, U1 STM8L101F2P3

Commit message: pcb: added JLC sn placeholder
Other:
- board text added: "JLCJLCJLCJLC"

Commit message: battery holder is now BH57A-5
Parts:
- BT1: footprint xmas_2021:HLD-001 -> xmas_2021:BH57A-5
- moved TP13 0.18 mm to (156.5, 118.0)
Connections:
- net /USR_BTN renamed Net-(SW1-Pad3)
Routing:
- net +BATT: track 63.7 -> 64.8 mm
Other:
- board text added: "CR2016"
- board text added: "v1.0"
