File: xmas_2021.kicad_pcb (KiCad board)
At the start: 2 copper layers, 41.4 x 69.4 mm, 36 parts, among them J1 SWIM, SW1 User, U1 STM8L101F2P3

Commit message: minor fixes
Other:
- board text added: "CR1620"
- board text removed: "CR2016"
